Commit message: GO: Add jetson & mount

File: urdf/components.urdf.xacro (robot description, xacro)
@@ -49,5 +49,6 @@
         ('DEV07T', 'dev07t'),
         ('DEV09', 'dev09'),
-        ('DEV10', 'dev10')
+        ('DEV10', 'dev10'),
+        ('DEV11', 'dev11')
       ])}" />
       <xacro:if value="${type in dev_models_dict}">

File: urdf/dev.urdf.xacro (robot description, xacro)
@@ -112,7 +112,16 @@
       <xacro:property name="rpy" value="0 0 0" scope="parent" />
       <xacro:property name="model_rpy" value="0 0 ${-pi/2.0}" scope="parent" />
-      <xacro:property name="collision_box_size" value="0.06 0.525 0.25"      scope="parent" />
+      <xacro:property name="collision_box_size" value="0.06 0.5 0.25"      scope="parent" />
+      <xacro:property name="collision_box_rpy"  value="0 0 0"      scope="parent" />
+      <xacro:property name="collision_box_xyz"  value="0 0 0.125"      scope="parent" />
+    </xacro:if>
+    <xacro:if value="${model == 'dev11'}">
+      <xacro:property name="parent_link" value="mount_link" scope="parent" />
+      <xacro:property name="xyz" value="-0.175 -0.117 -0.01"  scope="parent" />
+      <xacro:property name="rpy" value="0 0 ${-pi/2.0}" scope="parent" />
+      <xacro:property name="model_rpy" value="0 0 0" scope="parent" />
+      <xacro:property name="collision_box_size" value="0.35 0.02 0.02"      scope="parent" />
       <xacro:property name="collision_box_rpy"  value="0 0 ${-pi/2.0}"      scope="parent" />
-      <xacro:property name="collision_box_xyz"  value="0 0 0.125"      scope="parent" />
+      <xacro:property name="collision_box_xyz"  value="0.0 0.175 0.0"      scope="parent" />
     </xacro:if>
     <joint name="${model}_joint" type="fixed">
